File: MM Performer.kicad_sch (KiCad schematic)
At the start: 41 parts, among them IC1 68000D, J1 VCC, J2 GND, U1 MC68030RC, U2 MC68881FN-SOC, U3 ATF16V8BJ, U4 ATF16V8BJ, U5 ATF16V8BJ, U6 ATF16V8BJ, U7 ATF16V8BJ

Commit message: Draw PCB
Parts:
- removed unit 2 of U1
- added unit 2 of U1
- IC1: footprint Package_DIP:DIP-64_W22.86mm -> footprints:DIP-64_W22.86mm
- U3, U4, U5, U6: footprint footprints:PLCC-20_THT-Socket -> Package_LCC:PLCC-20_SMD-Socket
Connections:
- net GND: now also U1.C5 (GND@1), U1.C7 (GND@2), U1.C9 (GND@3), U1.E11 (GND@5), U1.E3 (GND@4), U1.F3 (GND@6), U1.G11 (GND@8), U1.G3 (GND@7), U1.J11 (GND@10), U1.J3 (GND@9), U1.L5 (GND@11), U1.L7 (GND@12), U1.L8 (GND@13), U1.L9 (GND@14)
- net VCC: now also U1.C6 (VCC@1), U1.D10 (VCC@3), U1.D4 (VCC@2), U1.F11 (VCC@5), U1.F2 (VCC@4), U1.H11 (VCC@7), U1.H3 (VCC@6), U1.K10 (VCC@9), U1.K4 (VCC@8), U1.L6 (VCC@10)

Commit message: Cleaning up the schematic
Connections:
- no-connect marks 30 -> 31
Other:
- note removed: "nc"
Changed lines of the file:
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@@
 		)
 	)
-	(text "nc"
-		(exclude_from_sim no)
-		(at 208.28 63.5 0)
-		(effects
-			(font
-				(size 1.778 1.5113)
-			)
-			(justify left bottom)
-		)
-	)
 	(junction
 		(at 401.32 274.32)
@@
 	)
 	(no_connect
+		(at 205.74 63.5)
+	)
+	(no_connect
 		(at 205.74 116.84)
 	)
@@
 	(wire
 		(pts
-			(xy 142.24 127) (xy 160.02 127)
-		)
-		(stroke
-			(width 0.1524)
-			(type solid)
-		)
-	)
-	(wire
-		(pts
 			(xy 378.46 271.78) (xy 378.46 274.32)
 		)
@@
 	(wire
 		(pts
+			(xy 142.24 127) (xy 152.4 127)
+		)
+		(stroke
+			(width 0)
+			(type default)
+		)
+	)
+	(wire
+		(pts
 			(xy 342.9 139.7) (xy 335.28 139.7)
 		)
@@
 	(wire
 		(pts
-			(xy 205.74 60.96) (xy 218.44 60.96)
+			(xy 205.74 60.96) (xy 222.25 60.96)
 		)
 		(stroke
@@
 	(wire
 		(pts
-			(xy 388.62 254) (xy 388.62 256.54)
+			(xy 241.3 114.3) (xy 256.54 114.3)
 		)
 		(stroke
-			(width 0)
-			(type default)
+			(width 0.1524)
+			(type solid)
 		)
 	)
 	(wire
 		(pts
-			(xy 81.28 320.04) (xy 81.28 318.77)
+			(xy 388.62 254) (xy 388.62 256.54)
 		)
 		(stroke
@@
 	(wire
 		(pts
-			(xy 328.93 254) (xy 328.93 256.54)
+			(xy 81.28 320.04) (xy 81.28 318.77)
 		)
 		(stroke
@@
 	(wire
 		(pts
-			(xy 243.84 114.3) (xy 256.54 114.3)
+			(xy 328.93 254) (xy 328.93 256.54)
 		)
 		(stroke
-			(width 0.1524)
-			(type solid)
+			(width 0)
+			(type default)
 		)
 	)
@@
 	)
 	(label "/AS_00"
-		(at 279.4 109.22 0)
+		(at 289.56 109.22 180)
 		(effects
 			(font
 				(size 1.2446 1.2446)
 			)
-			(justify left bottom)
+			(justify right bottom)
 		)
 	)
@@
 	)
 	(label "/FPUCS"
-		(at 208.28 53.34 0)
+		(at 218.44 53.34 180)
 		(effects
 			(font
 				(size 1.2446 1.2446)
 			)
-			(justify left bottom)
+			(justify right bottom)
 		)
 	)
 	(label "/CIIN"
-		(at 208.28 58.42 0)
+		(at 218.44 58.42 180)
 		(effects
 			(font
 				(size 1.2446 1.2446)
 			)
-			(justify left bottom)
+			(justify right bottom)
 		)
 	)
@@
 	)
 	(label "P2.A17"
-		(at 279.4 121.92 0)
+		(at 289.56 121.92 180)
 		(effects
 			(font
 				(size 1.2446 1.2446)
 			)
-			(justify left bottom)
+			(justify right bottom)
 		)
 	)
@@
 	)
 	(label "SM_CLK16"
-		(at 279.4 53.34 0)
+		(at 289.56 53.34 180)
 		(effects
 			(font
 				(size 1.2446 1.2446)
 			)
-			(justify left bottom)
+			(justify right bottom)
 		)
 	)
@@
 	)
 	(label "FPUCLK"
-		(at 142.24 116.84 0)
+		(at 152.4 116.84 180)
 		(effects
 			(font
 				(size 1.2446 1.2446)
 			)
-			(justify left bottom)
+			(justify right bottom)
 		)
 	)
@@
 		)
 	)
-	(label "/RESET_30"
-		(at 256.54 66.04 0)
-		(effects
-			(font
-				(size 1.016 1.016)
-			)
-			(justify left bottom)
-		)
-	)
 	(label "FC1"
 		(at 172.72 63.5 0)
@@
 	)
 	(label "/DTACK_SYS+EX"
-		(at 208.28 60.96 0)
+		(at 222.25 60.96 180)
 		(effects
 			(font
 				(size 1.2446 1.2446)
 			)
-			(justify left bottom)
+			(justify right bottom)
 		)
 	)
@@
 	)
 	(label "N$1"
-		(at 279.4 68.58 0)
+		(at 289.56 68.58 180)
 		(effects
 			(font
 				(size 1.2446 1.2446)
 			)
-			(justify left bottom)
+			(justify right bottom)
 		)
 	)
@@
 	)
 	(label "/DTACK_SYS+EX"
-		(at 243.84 114.3 0)
+		(at 241.3 114.3 0)
 		(effects
 			(font
@@
 	)
 	(label "CLK_30"
-		(at 144.78 127 0)
+		(at 152.4 127 180)
 		(effects
 			(font
 				(size 1.2446 1.2446)
 			)
-			(justify left bottom)
+			(justify right bottom)
 		)
 	)
 	(label "/BERR_30"
-		(at 279.4 66.04 0)
+		(at 289.56 66.04 180)
 		(effects
 			(font
 				(size 1.2446 1.2446)
 			)
-			(justify left bottom)
+			(justify right bottom)
 		)
 	)
@@
 		)
 	)
-	(label "/SCC.RW.DEC"
-		(at 238.76 68.58 0)
-		(effects
-			(font
-				(size 1.2446 1.2446)
-			)
-			(justify left bottom)
-		)
-	)
 	(label "/CIIN"
 		(at 172.72 119.38 0)
@@
 	)
 	(label "CLK_30"
-		(at 279.4 50.8 0)
+		(at 289.56 50.8 180)
 		(effects
 			(font
 				(size 1.2446 1.2446)
 			)
-			(justify left bottom)
+			(justify right bottom)
 		)
 	)
@@
 	)
 	(label "CDIS"
-		(at 279.4 63.5 0)
+		(at 289.56 63.5 180)
 		(effects
 			(font
 				(size 1.2446 1.2446)
 			)
-			(justify left bottom)
+			(justify right bottom)
 		)
 	)
@@
 	)
 	(label "A23"
-		(at 173.99 45.72 0)
+		(at 172.72 45.72 0)
 		(effects
 			(font
@@
 		)
 	)
-	(label "NOFC"
-		(at 243.84 106.68 180)
-		(effects
-			(font
-				(size 1.016 1.016)
-			)
-			(justify right bottom)
-		)
-	)
 	(label "/CIIN"
 		(at 327.66 76.2 0)
@@
 	)
 	(label "P3.B10"
-		(at 208.28 45.72 0)
+		(at 218.44 45.72 180)
 		(effects
 			(font
 				(size 1.2446 1.2446)
 			)
-			(justify left bottom)
+			(justify right bottom)
 		)
 	)
@@
 	)
 	(label "/EXT.DTK"
-		(at 208.28 66.04 0)
+		(at 218.44 66.04 180)
 		(effects
 			(font
 				(size 1.2446 1.2446)
 			)
-			(justify left bottom)
+			(justify right bottom)
 		)
 	)
@@
 	)
 	(label "/VMA"
-		(at 279.4 114.3 0)
+		(at 289.56 114.3 180)
 		(effects
 			(font
 				(size 1.2446 1.2446)
 			)
-			(justify left bottom)
+			(justify right bottom)
 		)
 	)
@@
 	)
 	(label "NOFC"
-		(at 208.28 50.8 0)
+		(at 218.44 50.8 180)
 		(effects
 			(font
 				(size 1.2446 1.2446)
 			)
-			(justify left bottom)
+			(justify right bottom)
 		)
 	)
 	(label "/DSACK1"
-		(at 279.4 124.46 0)
+		(at 289.56 124.46 180)
 		(effects
 			(font
 				(size 1.2446 1.2446)
 			)
-			(justify left bottom)
+			(justify right bottom)
 		)
 	)
@@
 	)
 	(label "AVEC"
-		(at 208.28 55.88 0)
+		(at 218.44 55.88 180)
 		(effects
 			(font
 				(size 1.2446 1.2446)
 			)
-			(justify left bottom)
+			(justify right bottom)
 		)
 	)
